Commit message: weak1:实现paxini和bulb的移植 增加task训练任务

File: assets/dexh13_right_description/urdf/dexh13_right_fix_path.urdf (robot description, URDF)
Before this commit: robot dexh13_right, 28 links, 27 joints
Links:
- link right_palm_link: geometry collision mesh filename=../meshes/right_palm_link.STL scale=0.1 0.1 0.1; visual mesh filename=../meshes/right_palm_link.STL
