Commit message: 修改paxini的urdf问题，缩小部分collision面积，修改部分杆的依赖关系，解决初始自碰撞导致的力矩过大问题。优化部分奖励参数，调整初始位置

File: assets/dexh13_right_description2/urdf/dexh13_right.urdf (robot description, URDF)
Before this commit: robot dexh13_right, 28 links, 27 joints
Links:
- link right_index_link_0: geometry collision mesh filename=package://dexh13_right_description/meshes/right_index_link_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; visual mesh filename=package://dexh13_right_description/meshes/right_index_link_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
- link right_index_link_1: geometry collision mesh filename=package://dexh13_right_description/meshes/right_index_link_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; visual mesh filename=package://dexh13_right_description/meshes/right_index_link_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
- link right_index_link_2: geometry collision mesh filename=package://dexh13_right_description/meshes/right_index_link_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; visual mesh filename=package://dexh13_right_description/meshes/right_index_link_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
- link right_index_link_3: geometry collision mesh filename=package://dexh13_right_description/meshes/right_index_link_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; visual mesh filename=package://dexh13_right_description/meshes/right_index_link_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
- link right_index_tactile_link_0: geometry collision mesh filename=package://dexh13_right_description/meshes/right_index_tacti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; visual mesh filename=package://dexh13_right_description/meshes/right_index_tacti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
- link right_index_tactile_link_1: geometry collision mesh filename=package://dexh13_right_description/meshes/right_index_tacti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; visual mesh filename=package://dexh13_right_description/meshes/right_index_tacti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
- link right_index_tactile_link_2: geometry collision mesh filename=package://dexh13_right_description/meshes/right_index_tacti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; visual mesh filename=package://dexh13_right_description/meshes/right_index_tacti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
- link right_middle_link_0: geometry collision mesh filename=package://dexh13_right_description/meshes/right_middle_link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; visual mesh filename=package://dexh13_right_description/meshes/right_middle_link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
- link right_middle_link_1: geometry collision mesh filename=package://dexh13_right_description/meshes/right_middle_link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; visual mesh filename=package://dexh13_right_description/meshes/right_middle_link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
- link right_middle_link_2: geometry collision mesh filename=package://dexh13_right_description/meshes/right_middle_link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; visual mesh filename=package://dexh13_right_description/meshes/right_middle_link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
- link right_middle_link_3: geometry collision mesh filename=package://dexh13_right_description/meshes/right_middle_link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; visual mesh filename=package://dexh13_right_description/meshes/right_middle_link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
- link right_middle_tactile_link_0: geometry collision mesh filename=package://dexh13_right_description/meshes/right_middle_tact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; visual mesh filename=package://dexh13_right_description/meshes/right_middle_tact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
- link right_middle_tactile_link_1: geometry collision mesh filename=package://dexh13_right_description/meshes/right_middle_tact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; visual mesh filename=package://dexh13_right_description/meshes/right_middle_tact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
- link right_middle_tactile_link_2: geometry collision mesh filename=package://dexh13_right_description/meshes/right_middle_tact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; visual mesh filename=package://dexh13_right_description/meshes/right_middle_tact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
- link right_palm_link: geometry collision mesh filename=package://dexh13_right_description/meshes/right_palm_link.S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; visual mesh filename=package://dexh13_right_description/meshes/right_palm_link.S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
- link right_ring_link_0: geometry collision mesh filename=package://dexh13_right_description/meshes/right_ring_link_0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; visual mesh filename=package://dexh13_right_description/meshes/right_ring_link_0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
- link right_ring_link_1: geometry collision mesh filename=package://dexh13_right_description/meshes/right_ring_link_1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; visual mesh filename=package://dexh13_right_description/meshes/right_ring_link_1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
- link right_ring_link_2: geometry collision mesh filename=package://dexh13_right_description/meshes/right_ring_link_2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; visual mesh filename=package://dexh13_right_description/meshes/right_ring_link_2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
- link right_ring_link_3: geometry collision mesh filename=package://dexh13_right_description/meshes/right_ring_link_3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; visual mesh filename=package://dexh13_right_description/meshes/right_ring_link_3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
- link right_ring_tactile_link_0: geometry collision mesh filename=package://dexh13_right_description/meshes/right_ring_tactil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; visual mesh filename=package://dexh13_right_description/meshes/right_ring_tactil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
- link right_ring_tactile_link_1: geometry collision mesh filename=package://dexh13_right_description/meshes/right_ring_tactil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; visual mesh filename=package://dexh13_right_description/meshes/right_ring_tactil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
- link right_ring_tactile_link_2: geometry collision mesh filename=package://dexh13_right_description/meshes/right_ring_tactil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; visual mesh filename=package://dexh13_right_description/meshes/right_ring_tactil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
- link right_thumb_link_0: geometry collision mesh filename=package://dexh13_right_description/meshes/right_thumb_link_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; visual mesh filename=package://dexh13_right_description/meshes/right_thumb_link_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
- link right_thumb_link_1: geometry collision mesh filename=package://dexh13_right_description/meshes/right_thumb_link_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; visual mesh filename=package://dexh13_right_description/meshes/right_thumb_link_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
- link right_thumb_link_2: geometry collision mesh filename=package://dexh13_right_description/meshes/right_thumb_link_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; visual mesh filename=package://dexh13_right_description/meshes/right_thumb_link_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
- link right_thumb_link_3: geometry collision mesh filename=package://dexh13_right_description/meshes/right_thumb_link_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; visual mesh filename=package://dexh13_right_description/meshes/right_thumb_link_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
- link right_thumb_tactile_link_0: geometry collision mesh filename=package://dexh13_right_description/meshes/right_thumb_tacti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; visual mesh filename=package://dexh13_right_description/meshes/right_thumb_tacti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
- link right_thumb_tactile_link_1: geometry collision mesh filename=package://dexh13_right_description/meshes/right_thumb_tacti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; visual mesh filename=package://dexh13_right_description/meshes/right_thumb_tacti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

File: assets/dexh13_right_description2/urdf/dexh13_right1.urdf (robot description, URDF)
Before this commit: robot dexh13_right, 28 links, 27 joints
Links:
- link right_index_link_1: geometry collision mesh filename=../meshes/right_index_link_1.STL; visual mesh filename=../meshes/right_index_link_1.STL
- link right_index_link_2: geometry collision mesh filename=../meshes/right_index_link_2.STL; visual mesh filename=../meshes/right_index_link_2.STL
- link right_index_link_3: geometry collision mesh filename=../meshes/right_index_link_3.STL; visual mesh filename=../meshes/right_index_link_3.STL
- link right_index_tactile_link_0: geometry collision mesh filename=../meshes/right_index_tactile_link_0.STL; visual mesh filename=../meshes/right_index_tactile_link_0.STL
- link right_index_tactile_link_1: geometry collision mesh filename=../meshes/right_index_tactile_link_1.STL; visual mesh filename=../meshes/right_index_tactile_link_1.STL
- link right_index_tactile_link_2: geometry collision mesh filename=../meshes/right_index_tactile_link_2.STL; visual mesh filename=../meshes/right_index_tactile_link_2.STL
- link right_middle_link_1: geometry collision mesh filename=../meshes/right_middle_link_1.STL; visual mesh filename=../meshes/right_middle_link_1.STL
- link right_middle_link_2: geometry collision mesh filename=../meshes/right_middle_link_2.STL; visual mesh filename=../meshes/right_middle_link_2.STL
- link right_middle_link_3: geometry collision mesh filename=../meshes/right_middle_link_3.STL; visual mesh filename=../meshes/right_middle_link_3.STL
- link right_middle_tactile_link_0: geometry collision mesh filename=../meshes/right_middle_tactile_link_0.STL; visual mesh filename=../meshes/right_middle_tactile_link_0.STL
- link right_middle_tactile_link_1: geometry collision mesh filename=../meshes/right_middle_tactile_link_1.STL; visual mesh filename=../meshes/right_middle_tactile_link_1.STL
- link right_middle_tactile_link_2: geometry collision mesh filename=../meshes/right_middle_tactile_link_2.STL; visual mesh filename=../meshes/right_middle_tactile_link_2.STL
- link right_palm_link: geometry collision mesh filename=../meshes/right_palm_link.STL; visual mesh filename=../meshes/right_palm_link.STL
- link right_ring_link_1: geometry collision mesh filename=../meshes/right_ring_link_1.STL; visual mesh filename=../meshes/right_ring_link_1.STL
- link right_ring_link_2: geometry collision mesh filename=../meshes/right_ring_link_2.STL; visual mesh filename=../meshes/right_ring_link_2.STL
- link right_ring_link_3: geometry collision mesh filename=../meshes/right_ring_link_3.STL; visual mesh filename=../meshes/right_ring_link_3.STL
- link right_ring_tactile_link_0: geometry collision mesh filename=../meshes/right_ring_tactile_link_0.STL; visual mesh filename=../meshes/right_ring_tactile_link_0.STL
- link right_ring_tactile_link_1: geometry collision mesh filename=../meshes/right_ring_tactile_link_1.STL; visual mesh filename=../meshes/right_ring_tactile_link_1.STL
- link right_ring_tactile_link_2: geometry collision mesh filename=../meshes/right_ring_tactile_link_2.STL; visual mesh filename=../meshes/right_ring_tactile_link_2.STL
- link right_thumb_link_2: geometry collision mesh filename=../meshes/right_thumb_link_2.STL; visual mesh filename=../meshes/right_thumb_link_2.STL
- link right_thumb_link_3: geometry collision mesh filename=../meshes/right_thumb_link_3.STL; visual mesh filename=../meshes/right_thumb_link_3.STL
- link right_thumb_tactile_link_0: geometry collision mesh filename=../meshes/right_thumb_tactile_link_0.STL; visual mesh filename=../meshes/right_thumb_tactile_link_0.STL
- link right_thumb_tactile_link_1: geometry collision mesh filename=../meshes/right_thumb_tactile_link_1.STL; visual mesh filename=../meshes/right_thumb_tactile_link_1.STL
